Commit message: commit

File: src/ros_06_urdf_rviz/urdf/urdf/demo05_test.urdf (robot description, URDF)
Before this commit: robot mycar, 6 links, 5 joints
Joints:
- joint left_wheel2base_link: origin xyz=0 0.1 -0.02 rpy=0 0 0 -> xyz=0 0.1 -0.0225 rpy=0 0 0
- joint right_wheel2base_link: origin xyz=0 -0.1 -0.02 rpy=0 0 0 -> xyz=0 -0.1 -0.0225 rpy=0 0 0
